File: keyboard.kicad_pcb (KiCad board)
At the start: 2 copper layers, 322.3 x 103.2 mm, 140 parts, among them J1 Conn_01x11, J2 Conn_01x11

Commit message: Add Adafruit feather wing socket. Version 0.1
Parts:
- J1: value Conn_01x11 -> Conn_01x16; footprint Connector_PinHeader_2.54mm:PinHeader_1x11_P2.54mm_Vertical -> Connector_PinSocket_2.54mm:PinSocket_1x16_P2.54mm_Vertical; moved to B.Cu
- J2: value Conn_01x11 -> Conn_01x12; footprint Connector_PinHeader_2.54mm:PinHeader_1x11_P2.54mm_Vertical -> Connector_PinSocket_2.54mm:PinSocket_1x12_P2.54mm_Vertical; moved to B.Cu
- moved J2 262.5 mm to (30.0, 16.3), turned to 90 degrees
- moved J1 250.5 mm to (40.2, 36.6), turned to 90 degrees
Connections:
- J1 pad 1: col0 -> Net-(J1-Pad1)
- J1 pad 10: col9 -> col13
- J1 pad 11: col10 -> col12
- J1 pad 2: col1 -> Net-(J1-Pad2)
- J1 pad 3: col2 -> Net-(J1-Pad3)
- J1 pad 4: col3 -> GND
- J1 pad 5: col4 -> col11
- J1 pad 6: col5 -> col10
- J1 pad 7: col6 -> col9
- J1 pad 8: col7 -> col15
- J1 pad 9: col8 -> col14
- J2 pad 1: col11 -> Net-(J2-Pad1)
- J2 pad 10: row4 -> col6
- J2 pad 11: Net-(J2-Pad11) -> col7
- J2 pad 2: col12 -> Net-(J2-Pad2)
- J2 pad 3: col13 -> Net-(J2-Pad3)
- J2 pad 4: col14 -> row4
- J2 pad 5: col15 -> row3
- J2 pad 6: row0 -> row2
- J2 pad 8: row2 -> row0
- J2 pad 9: row3 -> col5
Routing:
- net col15: track 86.5 -> 412.2 mm, vias 4 -> 1
- net col0: track 372.4 -> 93.8 mm
- net col1: track 360.7 -> 98.2 mm, vias 0 -> 1
- net col2: track 326.2 -> 93.5 mm, vias 4 -> 1
- net col14: track 119.1 -> 329.7 mm, vias 4 -> 1
- net row3: track 326.1 -> 509.3 mm, vias 1 -> 0
- net col13: track 160.5 -> 341.1 mm, vias 5 -> 1
- net col3: track 329.5 -> 165.4 mm, vias 6 -> 1
- net col12: track 159.1 -> 321.6 mm, vias 4 -> 2
- net row2: track 319.3 -> 468.3 mm, vias 0 -> 6
- net col4: track 283.7 -> 151.4 mm, vias 6 -> 1
- net col5: track 274.9 -> 166.0 mm, vias 4 -> 0
- net col11: track 176.2 -> 281.8 mm, vias 7 -> 1
- net row0: track 304.8 -> 400.9 mm, vias 0 -> 2
- net row1: track 305.2 -> 400.0 mm, vias 0 -> 8
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- added copper zone on B.Cu, net GND
- added copper zone on F.Cu, net GND
Other:
- board text added: "2021-02-07 Version: 0.1"
- board text removed: "col0"
- board text removed: "col11"
- board text removed: "row0"
- board text removed: "row4"
